Commit message: modified dimensions

File: Simulation/hand.urdf (robot description, URDF)
Before this commit: robot Hand, 13 links, 12 joints
Links:
- link arm: geometry visual mesh filename=meshes/arm_reduced.stl scale=.0005 .0005 .0015
- link index0: geometry visual mesh filename=meshes/finger_long_reduced.stl scale=.005 .005 .005
- link index1: geometry visual mesh filename=meshes/finger_long_reduced.stl scale=.005 .005 .005
- link little0: geometry visual mesh filename=meshes/finger_long_reduced.stl scale=.005 .005 .005
- link little1: geometry visual mesh filename=meshes/finger_short_reduced.stl scale=.005 .005 .005
- link middle0: geometry visual mesh filename=meshes/finger_long_reduced.stl scale=.005 .005 .005
- link middle1: geometry visual mesh filename=meshes/finger_long_reduced.stl scale=.005 .005 .005
- link palm: geometry visual mesh filename=meshes/palm_reduced.stl scale=.005 .005 .005
- link ring0: geometry visual mesh filename=meshes/finger_long_reduced.stl scale=.005 .005 .005
- link ring1: geometry visual mesh filename=meshes/finger_long_reduced.stl scale=.005 .005 .005
- link thumb0: geometry visual mesh filename=meshes/finger_long_reduced.stl scale=.005 .005 .005
- link thumb1: geometry visual mesh filename=meshes/finger_long_reduced.stl scale=.005 .005 .005
Joints:
- joint index_0_1: origin xyz=0 0 0.6 rpy=0 0 0 -> xyz=0 0 0.3 rpy=0 0 0
- joint indexpalm: origin xyz=-0.3 0 0.7 rpy=0 -0.1 0 -> xyz=-0.15 0 0.35 rpy=0 -0.1 0
- joint little_0_1: origin xyz=0 0 0.6 rpy=0 0 0 -> xyz=0 0 0.3 rpy=0 0 0
- joint littlepalm: origin xyz=1 0 0.4 rpy=0 0.5 0 -> xyz=0.5 0 0.2 rpy=0 0.5 0
- joint middle_0_1: origin xyz=0 0 0.6 rpy=0 0 0 -> xyz=0 0 0.3 rpy=0 0 0
- joint middlepalm: origin xyz=0.15 0 0.8 rpy=0 0 0 -> xyz=0.075 0 0.4 rpy=0 0 0
- joint ring_0_1: origin xyz=0 0 0.6 rpy=0 0 0 -> xyz=0 0 0.3 rpy=0 0 0
- joint ringpalm: origin xyz=0.6 0 0.7 rpy=0 0.2 0 -> xyz=0.3 0 0.35 rpy=0 0.2 0
- joint thumb_0_1: origin xyz=0 0 0.6 rpy=0 0 0 -> xyz=0 0 0.3 rpy=0 0 0
- joint thumbpalm: origin xyz=-0.4 0 -0.9 rpy=0 -0.80 0 -> xyz=-0.2 0 -0.45 rpy=0 -0.80 0
- joint wrist: origin xyz=-0.1 0 5 rpy=0 0 0 -> xyz=-0.05 0 2.5 rpy=0 0 0

Commit message: Arm swinging and dimension modification

File: Simulation/hand.urdf (robot description, URDF)
Before this commit: robot Hand, 13 links, 12 joints
Links:
- link arm: mass None -> 0.001; geometry visual mesh filename=meshes/arm_reduced.stl scale=4e-4 4e-4 1.2e-3
- link index0: mass None -> 0.0001
- link index1: mass None -> 0.0001
- link little0: mass None -> 0.0001
- link little1: mass None -> 0.0001
- link middle0: mass None -> 0.0001
- link middle1: mass None -> 0.0001
- link palm: mass None -> 0.0001
- link ring0: mass None -> 0.0001
- link ring1: mass None -> 0.0001
- link thumb0: mass None -> 0.0001
- link thumb1: mass None -> 0.0001
Joints:
- joint armbase: axis (none) -> 0 1 0; limit (none) -> effort=10 velocity=0.01; type fixed -> revolute
- joint wrist: origin xyz=-0.05 0 2.5 rpy=0 0 0 -> xyz=-0.05 0 2.1 rpy=0 0 0

Commit message: Wrist Movement

File: Simulation/hand.urdf (robot description, URDF)
Before this commit: robot Hand, 13 links, 12 joints
Links:
- link arm: mass 0.001 -> 0.002
Joints:
- joint indexpalm: origin xyz=-0.15 0 0.35 rpy=0 -0.1 0 -> xyz=-0.15 0 0.8 rpy=0 -0.1 0
- joint littlepalm: origin xyz=0.5 0 0.2 rpy=0 0.5 0 -> xyz=0.5 0 0.65 rpy=0 0.5 0
- joint middlepalm: origin xyz=0.075 0 0.4 rpy=0 0 0 -> xyz=0.075 0 0.85 rpy=0 0 0
- joint ringpalm: origin xyz=0.3 0 0.35 rpy=0 0.2 0 -> xyz=0.3 0 0.8 rpy=0 0.2 0
- joint thumbpalm: origin xyz=-0.2 0 -0.45 rpy=0 -0.80 0 -> xyz=-0.2 0 0 rpy=0 -0.80 0
- joint wrist: axis (none) -> 0 1 0; limit (none) -> effort=10 velocity=1; origin xyz=-0.05 0 2.1 rpy=0 0 0 -> xyz=-0.05 0 1.7 rpy=0 0 0; type fixed -> revolute
